Commit message: Rudimentary Spiderbot body created

File: body.urdf (robot description, URDF)
Before this commit: robot robot, 9 links, 8 joints
Links:
- removed link BackLeg
- removed link BackLowerLeg
- removed link FrontLeg
- removed link FrontLowerLeg
- removed link LeftLeg
- removed link LeftLowerLeg
- removed link RightLeg
- removed link RightLowerLeg
- added link LeftLeg1, mass 1; collision box size=1 0.2 0.2; visual box size=1 0.2 0.2
- added link LeftLeg2, mass 1; collision box size=1 0.2 0.2; visual box size=1 0.2 0.2
- added link LeftLeg3, mass 1; collision box size=1 0.2 0.2; visual box size=1 0.2 0.2
- added link LeftLeg4, mass 1; collision box size=1 0.2 0.2; visual box size=1 0.2 0.2
- added link LeftLowerLeg1, mass 1; collision box size=0.2 0.2 1; visual box size=0.2 0.2 1
- added link LeftLowerLeg2, mass 1; collision box size=0.2 0.2 1; visual box size=0.2 0.2 1
- added link LeftLowerLeg3, mass 1; collision box size=0.2 0.2 1; visual box size=0.2 0.2 1
- added link LeftLowerLeg4, mass 1; collision box size=0.2 0.2 1; visual box size=0.2 0.2 1
- added link RightLeg1, mass 1; collision box size=1 0.2 0.2; visual box size=1 0.2 0.2
- added link RightLeg2, mass 1; collision box size=1 0.2 0.2; visual box size=1 0.2 0.2
- added link RightLeg3, mass 1; collision box size=1 0.2 0.2; visual box size=1 0.2 0.2
- added link RightLeg4, mass 1; collision box size=1 0.2 0.2; visual box size=1 0.2 0.2
- added link RightLowerLeg1, mass 1; collision box size=0.2 0.2 1; visual box size=0.2 0.2 1
- added link RightLowerLeg2, mass 1; collision box size=0.2 0.2 1; visual box size=0.2 0.2 1
- added link RightLowerLeg3, mass 1; collision box size=0.2 0.2 1; visual box size=0.2 0.2 1
- added link RightLowerLeg4, mass 1; collision box size=0.2 0.2 1; visual box size=0.2 0.2 1
- link Torso: geometry collision box size=1 2 1; visual box size=1 2 1
Joints:
- removed joint BackLeg_BackLowerLeg
- removed joint FrontLeg_FrontLowerLeg
- removed joint LeftLeg_LeftLowerLeg
- removed joint RightLeg_RightLowerLeg
- removed joint Torso_BackLeg
- removed joint Torso_FrontLeg
- removed joint Torso_LeftLeg
- removed joint Torso_RightLeg
- added joint LeftLeg_LeftLowerLeg1: type revolute, parent LeftLeg1, child LeftLowerLeg1, origin xyz=-1 0 0 rpy=0 0 0, axis 0 1 0, limit lower=-3.14159 upper=3.14159 effort=0.0 velocity=0.0
- added joint LeftLeg_LeftLowerLeg2: type revolute, parent LeftLeg2, child LeftLowerLeg2, origin xyz=-1 0 0 rpy=0 0 0, axis 0 1 0, limit lower=-3.14159 upper=3.14159 effort=0.0 velocity=0.0
- added joint LeftLeg_LeftLowerLeg3: type revolute, parent LeftLeg3, child LeftLowerLeg3, origin xyz=-1 0 0 rpy=0 0 0, axis 0 1 0, limit lower=-3.14159 upper=3.14159 effort=0.0 velocity=0.0
- added joint LeftLeg_LeftLowerLeg4: type revolute, parent LeftLeg4, child LeftLowerLeg4, origin xyz=-1 0 0 rpy=0 0 0, axis 0 1 0, limit lower=-3.14159 upper=3.14159 effort=0.0 velocity=0.0
- added joint RightLeg_RightLowerLeg1: type revolute, parent RightLeg1, child RightLowerLeg1, origin xyz=1 0 0 rpy=0 0 0, axis 0 1 0, limit lower=-3.14159 upper=3.14159 effort=0.0 velocity=0.0
- added joint RightLeg_RightLowerLeg2: type revolute, parent RightLeg2, child RightLowerLeg2, origin xyz=1 0 0 rpy=0 0 0, axis 0 1 0, limit lower=-3.14159 upper=3.14159 effort=0.0 velocity=0.0
- added joint RightLeg_RightLowerLeg3: type revolute, parent RightLeg3, child RightLowerLeg3, origin xyz=1 0 0 rpy=0 0 0, axis 0 1 0, limit lower=-3.14159 upper=3.14159 effort=0.0 velocity=0.0
- added joint RightLeg_RightLowerLeg4: type revolute, parent RightLeg4, child RightLowerLeg4, origin xyz=1 0 0 rpy=0 0 0, axis 0 1 0, limit lower=-3.14159 upper=3.14159 effort=0.0 velocity=0.0
- added joint Torso_LeftLeg1: type revolute, parent Torso, child LeftLeg1, origin xyz=-0.5 0 1 rpy=0 0 0, axis 0 1 0, limit lower=-3.14159 upper=3.14159 effort=0.0 velocity=0.0
- added joint Torso_LeftLeg2: type revolute, parent Torso, child LeftLeg2, origin xyz=-0.5 0 1 rpy=0 0 0, axis 0 1 0, limit lower=-3.14159 upper=3.14159 effort=0.0 velocity=0.0
- added joint Torso_LeftLeg3: type revolute, parent Torso, child LeftLeg3, origin xyz=-0.5 0 1 rpy=0 0 0, axis 0 1 0, limit lower=-3.14159 upper=3.14159 effort=0.0 velocity=0.0
- added joint Torso_LeftLeg4: type revolute, parent Torso, child LeftLeg4, origin xyz=-0.5 0 1 rpy=0 0 0, axis 0 1 0, limit lower=-3.14159 upper=3.14159 effort=0.0 velocity=0.0
- added joint Torso_RightLeg1: type revolute, parent Torso, child RightLeg1, origin xyz=0.5 0 1 rpy=0 0 0, axis 0 1 0, limit lower=-3.14159 upper=3.14159 effort=0.0 velocity=0.0
- added joint Torso_RightLeg2: type revolute, parent Torso, child RightLeg2, origin xyz=0.5 0 1 rpy=0 0 0, axis 0 1 0, limit lower=-3.14159 upper=3.14159 effort=0.0 velocity=0.0
- added joint Torso_RightLeg3: type revolute, parent Torso, child RightLeg3, origin xyz=0.5 0 1 rpy=0 0 0, axis 0 1 0, limit lower=-3.14159 upper=3.14159 effort=0.0 velocity=0.0
- added joint Torso_RightLeg4: type revolute, parent Torso, child RightLeg4, origin xyz=0.5 0 1 rpy=0 0 0, axis 0 1 0, limit lower=-3.14159 upper=3.14159 effort=0.0 velocity=0.0

Commit message: Milestone 1: Successfully met base conditions for Spiderbot

File: body.urdf (robot description, URDF)
Before this commit: robot robot, 17 links, 16 joints
Joints:
- joint LeftLeg_LeftLowerLeg1: axis 0 1 0 -> 1 1 0 
- joint LeftLeg_LeftLowerLeg2: axis 0 1 0 -> 1 1 0 
- joint LeftLeg_LeftLowerLeg3: axis 0 1 0 -> 1 1 0 
- joint LeftLeg_LeftLowerLeg4: axis 0 1 0 -> 1 1 0 
- joint RightLeg_RightLowerLeg1: axis 0 1 0 -> 1 1 0 
- joint RightLeg_RightLowerLeg2: axis 0 1 0 -> 1 1 0 
- joint RightLeg_RightLowerLeg3: axis 0 1 0 -> 1 1 0 
- joint RightLeg_RightLowerLeg4: axis 0 1 0 -> 1 1 0 
- joint Torso_LeftLeg1: axis 0 1 0 -> 1 1 0 
- joint Torso_LeftLeg2: axis 0 1 0 -> 1 1 0 
- joint Torso_LeftLeg3: axis 0 1 0 -> 1 1 0 
- joint Torso_LeftLeg4: axis 0 1 0 -> 1 1 0 
- joint Torso_RightLeg1: axis 0 1 0 -> 1 1 0 
- joint Torso_RightLeg2: axis 0 1 0 -> 1 1 0 
- joint Torso_RightLeg3: axis 0 1 0 -> 1 1 0 
- joint Torso_RightLeg4: axis 0 1 0 -> 1 1 0 

Commit message: Milestone 02

File: body.urdf (robot description, URDF)
Before this commit: robot robot, 17 links, 16 joints
Joints:
- joint LeftLeg_LeftLowerLeg1: axis 1 1 0  -> 0 1 0 
- joint LeftLeg_LeftLowerLeg2: axis 1 1 0  -> 0 1 0 
- joint LeftLeg_LeftLowerLeg3: axis 1 1 0  -> 0 1 0 
- joint LeftLeg_LeftLowerLeg4: axis 1 1 0  -> 0 1 0 
- joint RightLeg_RightLowerLeg1: axis 1 1 0  -> 0 1 0 
- joint RightLeg_RightLowerLeg2: axis 1 1 0  -> 0 1 0 
- joint RightLeg_RightLowerLeg3: axis 1 1 0  -> 0 1 0 
- joint RightLeg_RightLowerLeg4: axis 1 1 0  -> 0 1 0 
- joint Torso_LeftLeg1: axis 1 1 0  -> 0 1 0 
- joint Torso_LeftLeg2: axis 1 1 0  -> 0 1 0 
- joint Torso_LeftLeg3: axis 1 1 0  -> 0 1 0 
- joint Torso_LeftLeg4: axis 1 1 0  -> 0 1 0 
- joint Torso_RightLeg1: axis 1 1 0  -> 0 1 0 
- joint Torso_RightLeg2: axis 1 1 0  -> 0 1 0 
- joint Torso_RightLeg3: axis 1 1 0  -> 0 1 0 
- joint Torso_RightLeg4: axis 1 1 0  -> 0 1 0 
